File: ledfoot.kicad_sch (KiCad schematic)
At the start: 24 parts, among them J1 1729144, J2 54-00167, J3 Conn_01x12_Pin, SW1 SW_Push, SW2 SW_Push, U1 MP1584EN, U2 SN74LVC1T45DBV

Commit message: Correct project naming
Other:
- title: LED Foot -> LEDFoot
Changed lines of the file:
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@@
 	(paper "USLetter")
 	(title_block
-		(title "LED Foot")
+		(title "LEDFoot")
 		(date "2025-01-03")
 		(rev "1")
@@
 		)
 		(instances
-			(project "ws2815_surface"
+			(project "ledfoot"
 				(path "/dd2ab11b-80e0-45f1-9b50-8fbc67a3597c"
 					(reference "SW2")
@@
 		)
 		(instances
-			(project "ws2815_surface"
+			(project "ledfoot"
 				(path "/dd2ab11b-80e0-45f1-9b50-8fbc67a3597c"
 					(reference "#PWR011")
@@
 		)
 		(instances
-			(project "ws2815_surface"
+			(project "ledfoot"
 				(path "/dd2ab11b-80e0-45f1-9b50-8fbc67a3597c"
 					(reference "#PWR010")
@@
 		)
 		(instances
-			(project "ws2815_surface"
+			(project "ledfoot"
 				(path "/dd2ab11b-80e0-45f1-9b50-8fbc67a3597c"
 					(reference "#PWR03")
@@
 		)
 		(instances
-			(project "ws2815_surface"
+			(project "ledfoot"
 				(path "/dd2ab11b-80e0-45f1-9b50-8fbc67a3597c"
 					(reference "C7")
@@
 		)
 		(instances
-			(project "ws2815_surface"
+			(project "ledfoot"
 				(path "/dd2ab11b-80e0-45f1-9b50-8fbc67a3597c"
 					(reference "#PWR05")
@@
 		)
 		(instances
-			(project "ws2815_surface"
+			(project "ledfoot"
 				(path "/dd2ab11b-80e0-45f1-9b50-8fbc67a3597c"
 					(reference "#PWR04")
@@
 		)
 		(instances
-			(project "ws2815_surface"
+			(project "ledfoot"
 				(path "/dd2ab11b-80e0-45f1-9b50-8fbc67a3597c"
 					(reference "R5")
@@
 		)
 		(instances
-			(project "ws2815_surface"
+			(project "ledfoot"
 				(path "/dd2ab11b-80e0-45f1-9b50-8fbc67a3597c"
 					(reference "#PWR014")
@@
 		)
 		(instances
-			(project "ws2815_surface"
+			(project "ledfoot"
 				(path "/dd2ab11b-80e0-45f1-9b50-8fbc67a3597c"
 					(reference "#FLG02")
@@
 		)
 		(instances
-			(project "ws2815_surface"
+			(project "ledfoot"
 				(path "/dd2ab11b-80e0-45f1-9b50-8fbc67a3597c"
 					(reference "#PWR08")
@@
 		)
 		(instances
-			(project "ws2815_surface"
+			(project "ledfoot"
 				(path "/dd2ab11b-80e0-45f1-9b50-8fbc67a3597c"
 					(reference "C6")
@@
 		)
 		(instances
-			(project "ws2815_surface"
+			(project "ledfoot"
 				(path "/dd2ab11b-80e0-45f1-9b50-8fbc67a3597c"
 					(reference "C4")
@@
 		)
 		(instances
-			(project "ws2815_surface"
+			(project "ledfoot"
 				(path "/dd2ab11b-80e0-45f1-9b50-8fbc67a3597c"
 					(reference "#FLG03")
@@
 		)
 		(instances
-			(project "ws2815_surface"
+			(project "ledfoot"
 				(path "/dd2ab11b-80e0-45f1-9b50-8fbc67a3597c"
 					(reference "#PWR012")
@@
 		)
 		(instances
-			(project "ws2815_surface"
+			(project "ledfoot"
 				(path "/dd2ab11b-80e0-45f1-9b50-8fbc67a3597c"
 					(reference "#PWR07")
@@
 		)
 		(instances
-			(project "ws2815_surface"
+			(project "ledfoot"
 				(path "/dd2ab11b-80e0-45f1-9b50-8fbc67a3597c"
 					(reference "#PWR013")
@@
 		)
 		(instances
-			(project "ws2815_surface"
+			(project "ledfoot"
 				(path "/dd2ab11b-80e0-45f1-9b50-8fbc67a3597c"
 					(reference "R4")
@@
 		)
 		(instances
-			(project "ws2815_surface"
+			(project "ledfoot"
 				(path "/dd2ab11b-80e0-45f1-9b50-8fbc67a3597c"
 					(reference "#PWR06")
@@
 		)
 		(instances
-			(project "ws2815_surface"
+			(project "ledfoot"
 				(path "/dd2ab11b-80e0-45f1-9b50-8fbc67a3597c"
 					(reference "#PWR09")

Commit message: Revision 2 ready for production
Parts:
- removed 1: U?, Custom:WeAct-ESP32C3CoreBoard, symbol custom:ESP32-C3-WeAct-CH57xCH58xCoreBoard
- removed J3: Conn_01x12_Pin, Connector_PinHeader_2.54mm:PinHeader_1x12_P2.54mm_Vertical, symbol Connector:Conn_01x12_Pin
- removed SW2: SW_Push, Button_Switch_SMD:SW_SPST_PTS645, symbol Switch:SW_Push
- added C8: 0.1µF, Capacitor_SMD:C_0603_1608Metric, symbol Device:C
- added D3: SS34, Diode_SMD:D_SMA, symbol Diode:SS34
- added J3: Conn_02x05_Counter_Clockwise, Connector_PinHeader_2.54mm:PinHeader_2x06_P2.54mm_Vertical_SMD, symbol Connector_Generic:Conn_02x06_Odd_Even
- added MK1: SPK0641HT4H-1, MIC_SPK0641HT4H-1:MIC_SPK0641HT4H-1, symbol SPK0641HT4H-1:SPK0641HT4H-1
- added Q1: SIRA20DP-T1-RE3, POWERPAK_SO-8_SINGLE_VIS:POWERPAK_SO-8_SINGLE_VIS, symbol SiRA20DP_T1_RE3:SIRA20DP-T1-RE3
- added R6: 1MΩ, Resistor_SMD:R_0603_1608Metric, symbol Device:R_US
- added R7: 10Ω, Resistor_SMD:R_0603_1608Metric, symbol Device:R_US
- added U3: ~, Tenstar-ESP32:Tenstar-ESP32-S3-SuperMini-EdgeOnly, symbol Tenstar-ESP32:Tenstar-ESP32-S3-SuperMini-EdgeOnly
- C1: footprint Capacitor_THT:CP_Radial_D10.0mm_P5.00mm -> Capacitor_THT:CP_Radial_D8.0mm_P3.50mm
- C3, C4, C5: footprint Capacitor_SMD:C_0805_2012Metric -> Capacitor_SMD:C_0603_1608Metric
- F1: value 8A (RUEF800) -> RUEF800 (8A); footprint footprints:FUSRR505W81L660T250H1360 -> RUEF800:FUSE_RUEF800; symbol Device:Polyfuse -> RUEF800:RUEF800; Availability (none) -> In Stock; Check_prices (none) -> https://www.snapeda.com/parts/RUEF800/Littelfuse/view-part/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; Description_1 (none) -> Polymeric PTC Resettable Fuse 30V 8 A Ih Through Hole Radia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; MANUFACTURER (none) -> TE Connectivity; MF (none) -> Littelfuse Inc.; MP (none) -> RUEF800; Package (none) -> Radial Littelfuse; Price (none) -> None; SnapEDA_Link (none) -> https://www.snapeda.com/parts/RUEF800/Littelfuse/view-part/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
- J1: value 1729144 -> 1729144 (To WS2815s); footprint footprints:PHOENIX_1729144 -> Phoenix:PHOENIX_1729144
- J2: value 54-00167 -> 54-00167 (12V Barrel); footprint footprints:TENSILITY_54-00167 -> Tensility:TENSILITY_54-00167
- R1, R5: footprint Resistor_SMD:R_0805_2012Metric -> Resistor_SMD:R_0603_1608Metric
- R2: value 10kΩ -> 100kΩ; footprint Resistor_SMD:R_0805_2012Metric -> Resistor_SMD:R_0603_1608Metric
- R3: value 3.3kΩ -> 43kΩ; footprint Resistor_SMD:R_0805_2012Metric -> Resistor_SMD:R_0603_1608Metric
- R4: value 10kΩ -> 8.2kΩ; footprint Resistor_SMD:R_0805_2012Metric -> Resistor_SMD:R_0603_1608Metric
- U1: footprint Custom:SOIC127P600X170-9N -> MP1584EN:SOIC127P600X170-9N
Connections:
- net +12V: now also F1.2; no longer F1.1
- net 12V: now also F1.1, J3.10 (Pin_10); no longer F1.2, R2.1
- net 3V3: now also C8.1, J3.8 (Pin_8), MK1.4 (VDD), U3.16 (3V3)
- net 3V3_SIG: now also U3.7 (GP5)
- net 5V: now also J3.9 (Pin_9), U3.18 (5V)
- net GND: now also R2.1, D3.2 (A), J3.11 (Pin_11), Q1.1, Q1.2, Q1.3, R6.2, U3.17 (GND); no longer C6.2, C7.2, J1.4, U2.2 (GND)
- net at C5.2, L1.1, U1.1 (SW): now also D3.1 (K)
- net at R2.2: now also U1.6 (FREQ); no longer U1.2 (EN)
- net at SW1.1: now also U3.12 (GP10)
- new net: Q1.4, R7.2
- new net LEDS_EN: R6.1, R7.1, U3.6 (GP4)
- new net MIC_CLK: MK1.2 (CLOCK), U3.5 (GP3)
- new net MIC_DATA: MK1.1 (DATA), U3.4 (GP2)
- new net PIN1: J3.1 (Pin_1), U3.1 (TX)
- new net PIN2: J3.2 (Pin_2), U3.2 (RX)
- new net PIN3: J3.3 (Pin_3), U3.3 (GP1)
- new net PIN4: J3.4 (Pin_4), U3.15 (GP13)
- new net PIN5: J3.5 (Pin_5), U3.14 (GP12)
- new net PIN6: J3.6 (Pin_6), U3.13 (GP11)
- new net PIN7: J3.7 (Pin_7), U3.11 (GP9)
- new net SGND: C6.2, C7.2, C8.2, J1.4, J3.12 (Pin_12), MK1.3 (SELECT), MK1.5 (GND), MK1.6 (GND__1), MK1.7 (GND__2), MK1.8 (GND__3), Q1.5, U2.2 (GND)
- no-connect marks 12 -> 5
Other:
- moved on the sheet: C1, C2, C3, C4, C5, C6, C7, D1, D2, J1, J2, L1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

Commit message: Fix MP1584EN voltage divider swap
Parts:
- R3: value 43kΩ -> 8.2kΩ
- R4: value 8.2kΩ -> 43kΩ
Changed lines of the file:
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@@
 			)
 		)
-		(property "Value" "43kΩ"
+		(property "Value" "8.2kΩ"
 			(at 104.14 91.4399 0)
 			(effects
@@
 			)
 		)
-		(property "Value" "8.2kΩ"
+		(property "Value" "43kΩ"
 			(at 113.03 86.868 90)
 			(effects
